Commit message: update

File: src/ur_description/common.gazebo.xacro (robot description, xacro)
@@ -25,5 +25,5 @@
     <mu1>0.2</mu1>
     <mu2>0.2</mu2>
-    <material>Gazebo/Red</material>
+    <material>Gazebo/Green</material>
   </gazebo>
  <!-- camera -->

File: src/ur_description/ur5.urdf.xacro (robot description, xacro)
@@ -296,5 +296,5 @@
   <joint name="camera_joint" type="fixed">
     <axis xyz="0 1 0" />
-    <origin xyz="0.025 0.0 0" rpy="0 0 0"/>
+    <origin xyz="-0.02 0.0 0.055" rpy="0 0 0"/>
     <parent link="ee_link"/>
     <child link="camera_link"/>
@@ -313,5 +313,5 @@
 	<box size="${camera_link} ${camera_link} ${camera_link}"/>
       </geometry>
-      <material name="red"/>
+      <material name="green"/>
     </visual>
     <inertial>
